Commit message: fix urdf import bugs

File: gym_xarm/envs/urdf/my_cube.urdf (robot description, URDF)
Before this commit: robot cube, 1 links, 0 joints
Links:
- link baseLink: geometry collision box size=0.05 0.05 0.05; visual mesh filename=meshes/cube.obj scale=0.05 0.05 0.05

File: gym_xarm/envs/urdf/my_sphere.urdf (robot description, URDF)
Before this commit: robot urdf_robot, 1 links, 0 joints
Links:
- link base_link: geometry visual mesh filename=meshes/textured_sphere_smooth.obj scale=0.02 0.02 0.02

Commit message: change parameters

File: gym_xarm/envs/urdf/my_cube.urdf (robot description, URDF)
Before this commit: robot cube, 1 links, 0 joints
Links:
- link baseLink: mass 1 -> 0.01

File: gym_xarm/envs/urdf/xarm7.urdf (robot description, URDF)
Before this commit: robot xarm7_with_gripper, 18 links, 17 joints
Joints:
- joint drive_joint: limit lower=0 upper=0.85 effort=50 velocity=2 -> lower=0 upper=0.85 effort=5000 velocity=2
- joint left_finger_joint: limit lower=0 upper=0.85 effort=50 velocity=2 -> lower=0 upper=0.85 effort=5000 velocity=2
- joint left_inner_knuckle_joint: limit lower=0 upper=0.85 effort=50 velocity=2 -> lower=0 upper=0.85 effort=5000 velocity=2
- joint right_finger_joint: limit lower=0 upper=0.85 effort=50 velocity=2 -> lower=0 upper=0.85 effort=5000 velocity=2
- joint right_inner_knuckle_joint: limit lower=0 upper=0.85 effort=50 velocity=2 -> lower=0 upper=0.85 effort=5000 velocity=2
- joint right_outer_knuckle_joint: limit lower=0 upper=0.85 effort=50 velocity=2 -> lower=0 upper=0.85 effort=5000 velocity=2

Commit message: add a new gripper environment

File: gym_xarm/envs/urdf/my_cube.urdf (robot description, URDF)
Before this commit: robot cube, 1 links, 0 joints
Links:
- link baseLink: mass 0.01 -> 0.1

Commit message: fix pick and place

File: gym_xarm/envs/urdf/my_cube.urdf (robot description, URDF)
Before this commit: robot cube, 1 links, 0 joints
Links:
- link baseLink: mass 0.1 -> 0.5
